File: MODULES/motorized_potentiometer.sch (EAGLE design)
At the start: 4 parts, among them U1 MOTORIZEDPOT, U2 ADS1X15, U3 AT42QT1010, U4 TB6612FNG

Commit message: Fix paths
Parts:
- U1: value MOTORIZEDPOT -> MOTORIZEDPOT_MOTORIZEDPOT; device motorizedpot:MOTORIZEDPOT -> motorized_potentiometer:MOTORIZEDPOT_MOTORIZEDPOT
Changed lines of the file:
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@@
 </classes>
 <parts>
-<part name="U1" library="motorizedpot" deviceset="MOTORIZEDPOT" device=""/>
+<part name="U1" library="motorized_potentiometer" deviceset="MOTORIZEDPOT_MOTORIZEDPOT" device=""/>
 <part name="U2" library="ads1X15" deviceset="ADS1X15" device=""/>
 <part name="U3" library="AT42QT1010" deviceset="AT42QT1010" device=""/>
